File: labamp_SE_filter/labamp_SE_filter.kicad_sch (KiCad schematic)
At the start: 29 parts, among them J1 Conn_02x06_Odd_Even, J2 Conn_02x06_Odd_Even, J3 Conn_01x03, U1 ${SIM.PARAMS}

Commit message: SE filter routed 90%
Parts:
- added R1: R, Resistor_SMD:R_0603_1608Metric_Pad0.98x0.95mm_HandSolder, symbol Device:R
- renumbered Rout- to Rout-1, Rout to Rout1
Connections:
- net in-: now also R1.2
- net at C9.1, Ra1.1, Rb1.2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: now also R1.1
Other:
- moved on the sheet: Ra1, Rb1, Z6, Z7, Z8

Commit message: Finished routing
Parts:
- U1: value ${SIM.PARAMS} -> ~; footprint SOT-23-5 -> Package_TO_SOT_SMD:SOT-23-5
- renumbered Rout-1 to R2, Rout1 to R3
Changed lines of the file:
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@@
 		(on_board yes)
 		(dnp no)
-		(property "Reference" "Rout1"
+		(property "Reference" "R3"
 			(at 220.98 87.63 90)
 			(effects
@@
 			(project "labamp_SE_filter"
 				(path "/a0c99055-08c7-4e05-9803-96c7ce32a2b2"
-					(reference "Rout1")
+					(reference "R3")
 					(unit 1)
 				)
@@
 		(on_board yes)
 		(dnp no)
-		(property "Reference" "Rout-1"
+		(property "Reference" "R2"
 			(at 220.98 95.25 90)
 			(effects
@@
 			(project "labamp_SE_filter"
 				(path "/a0c99055-08c7-4e05-9803-96c7ce32a2b2"
-					(reference "Rout-1")
+					(reference "R2")
 					(unit 1)
 				)
@@
 			)
 		)
-		(property "Value" "${SIM.PARAMS}"
+		(property "Value" "~"
 			(at 166.37 90.7349 0)
 			(effects
@@
 			)
 		)
-		(property "Footprint" "SOT-23-5"
+		(property "Footprint" "Package_TO_SOT_SMD:SOT-23-5"
 			(at 158.75 93.98 0)
 			(effects
